File: nRF24-MultiPro.sch (EAGLE design)
At the start: 13 parts, among them IC1 SPX3819, J1 22-27-2051-05, Q1 BSS123

Commit message: v1.1 pcb
- 470pF for low noise
- slightly rearanged SMDs
- manualy traced some wires
- GND and VCC upped to 8mil
- added logo
Parts:
- added C2: 470pF, resistor:C-EUC0805
- C1: value (none) -> 2.2uF
Connections:
- new net N$14: C2.1, IC1.BYP
- net GND: now also C2.2
Other:
- note added: "38-00-1395"
- note added: "Arduino Pro Mini 3v3 16M"
- moved on the sheet: IC1
Changed lines of the file:
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@@
 <?xml version="1.0" encoding="utf-8"?>
 <!DOCTYPE eagle SYSTEM "eagle.dtd">
-<eagle version="7.5.0">
+<eagle version="7.6.0">
 <drawing>
 <settings>
@@
 <parts>
 <part name="JP1" library="pinhead" deviceset="PINHD-2X4" device=""/>
-<part name="C1" library="resistor" deviceset="CPOL-EU" device="A/3216-18W"/>
+<part name="C1" library="resistor" deviceset="CPOL-EU" device="A/3216-18W" value="2.2uF"/>
 <part name="R1" library="resistor" deviceset="R-EU_" device="R0805" value="10k"/>
 <part name="IC1" library="v-reg-micrel" deviceset="MIC5219XX" device="" value="SPX3819"/>
@@
 <part name="R5" library="resistor" deviceset="R-EU_" device="R0805" value="1k"/>
 <part name="GND1" library="supply1" deviceset="GND" device=""/>
+<part name="C2" library="resistor" deviceset="C-EU" device="C0805" value="470pF"/>
 </parts>
 <sheets>
 <sheet>
 <plain>
+<text x="142.24" y="71.12" size="1.778" layer="91">Arduino Pro Mini
+3v3 16M</text>
+<text x="7.112" y="34.29" size="1.778" layer="91">38-00-1395</text>
 </plain>
 <instances>
@@
 <instance part="C1" gate="G$1" x="81.28" y="53.34"/>
 <instance part="R1" gate="G$1" x="91.44" y="86.36" rot="R90"/>
-<instance part="IC1" gate="G1" x="66.04" y="55.88"/>
-<instance part="J1" gate="-1" x="17.78" y="38.1" rot="R180"/>
+<instance part="IC1" gate="G1" x="66.04" y="60.96" smashed="yes">
+<attribute name="NAME" x="58.42" y="69.85" size="1.778" layer="95"/>
+<attribute name="VALUE" x="63.5" y="62.484" size="1.778" layer="96"/>
+</instance>
+<instance part="J1" gate="-1" x="17.78" y="38.1" smashed="yes" rot="R180">
+<attribute name="NAME" x="15.24" y="38.862" size="1.524" layer="95" rot="R180"/>
+</instance>
 <instance part="J1" gate="-2" x="17.78" y="43.18" rot="R180"/>
 <instance part="J1" gate="-3" x="17.78" y="48.26" rot="R180"/>
@@
 <instance part="R5" gate="G$1" x="50.8" y="25.4" rot="R270"/>
 <instance part="GND1" gate="1" x="76.2" y="35.56"/>
+<instance part="C2" gate="G$1" x="50.8" y="50.8"/>
 </instances>
 <busses>
@@
 <pinref part="J1" gate="-3" pin="S"/>
 <wire x1="20.32" y1="48.26" x2="33.02" y2="48.26" width="0.1524" layer="91"/>
-<wire x1="33.02" y1="48.26" x2="33.02" y2="55.88" width="0.1524" layer="91"/>
+<wire x1="33.02" y1="48.26" x2="33.02" y2="60.96" width="0.1524" layer="91"/>
 <pinref part="IC1" gate="G1" pin="IN"/>
-<wire x1="33.02" y1="55.88" x2="33.02" y2="60.96" width="0.1524" layer="91"/>
-<wire x1="33.02" y1="60.96" x2="55.88" y2="60.96" width="0.1524" layer="91"/>
+<wire x1="33.02" y1="60.96" x2="33.02" y2="66.04" width="0.1524" layer="91"/>
+<wire x1="33.02" y1="66.04" x2="55.88" y2="66.04" width="0.1524" layer="91"/>
 <pinref part="IC1" gate="G1" pin="EN"/>
-<wire x1="55.88" y1="55.88" x2="33.02" y2="55.88" width="0.1524" layer="91"/>
-<junction x="33.02" y="55.88"/>
+<wire x1="55.88" y1="60.96" x2="33.02" y2="60.96" width="0.1524" layer="91"/>
+<junction x="33.02" y="60.96"/>
 </segment>
 </net>
@@
 <net name="N$4" class="0">
 <segment>
-<pinref part="IC1" gate="G1" pin="OUT"/>
 <pinref part="C1" gate="G$1" pin="+"/>
 <wire x1="91.44" y1="60.96" x2="81.28" y2="60.96" width="0.1524" layer="91"/>
-<wire x1="81.28" y1="60.96" x2="76.2" y2="60.96" width="0.1524" layer="91"/>
 <wire x1="81.28" y1="55.88" x2="81.28" y2="60.96" width="0.1524" layer="91"/>
-<junction x="81.28" y="60.96"/>
 <pinref part="R1" gate="G$1" pin="1"/>
 <wire x1="91.44" y1="81.28" x2="91.44" y2="60.96" width="0.1524" layer="91"/>
@@
 <wire x1="50.8" y1="40.64" x2="50.8" y2="30.48" width="0.1524" layer="91"/>
 <junction x="101.6" y="40.64"/>
+<pinref part="IC1" gate="G1" pin="OUT"/>
+<wire x1="81.28" y1="60.96" x2="81.28" y2="66.04" width="0.1524" layer="91"/>
+<wire x1="81.28" y1="66.04" x2="76.2" y2="66.04" width="0.1524" layer="91"/>
+<junction x="81.28" y="60.96"/>
 </segment>
 </net>
@@
 <segment>
 <pinref part="J1" gate="-2" pin="S"/>
-<wire x1="20.32" y1="43.18" x2="60.96" y2="43.18" width="0.1524" layer="91"/>
+<wire x1="20.32" y1="43.18" x2="50.8" y2="43.18" width="0.1524" layer="91"/>
 <pinref part="IC1" gate="G1" pin="GND"/>
+<wire x1="50.8" y1="43.18" x2="60.96" y2="43.18" width="0.1524" layer="91"/>
 <wire x1="60.96" y1="43.18" x2="68.58" y2="43.18" width="0.1524" layer="91"/>
-<wire x1="68.58" y1="43.18" x2="68.58" y2="45.72" width="0.1524" layer="91"/>
+<wire x1="68.58" y1="43.18" x2="68.58" y2="50.8" width="0.1524" layer="91"/>
 <pinref part="JP1" gate="A" pin="1"/>
 <wire x1="76.2" y1="20.32" x2="68.58" y2="20.32" width="0.1524" layer="91"/>
@@
 <wire x1="76.2" y1="38.1" x2="76.2" y2="43.18" width="0.1524" layer="91"/>
 <junction x="76.2" y="43.18"/>
+<pinref part="C2" gate="G$1" pin="2"/>
+<wire x1="50.8" y1="45.72" x2="50.8" y2="43.18" width="0.1524" layer="91"/>
+<junction x="50.8" y="43.18"/>
 </segment>
 </net>
@@
 </segment>
 </net>
+<net name="N$14" class="0">
+<segment>
+<pinref part="C2" gate="G$1" pin="1"/>
+<pinref part="IC1" gate="G1" pin="BYP"/>
+<wire x1="50.8" y1="53.34" x2="50.8" y2="55.88" width="0.1524" layer="91"/>
+<wire x1="50.8" y1="55.88" x2="55.88" y2="55.88" width="0.1524" layer="91"/>
+</segment>
+</net>
 </nets>
 </sheet>
@@
 </schematic>
 </drawing>
+<compatibility>
+<note version="6.3" minversion="6.2.2" severity="warning">
+Since Version 6.2.2 text objects can contain more than one line,
+which will not be processed correctly with this version.
+</note>
+</compatibility>
 </eagle>
